File: kicad/lipo_arduino_core.sch (KiCad schematic (older format))
At the start: 26 parts, among them CON1 LIPO_BAT, CON2 USB-MINI-B, CON3 ICSP, SW1 SPDT, SW2 SPST, U1 MCP73831, U2 MIC5219, U3 ATMEGA32U4

Commit message: fixed bugs in schematic, created parts list
Parts:
- added R4, R5: 22, ~, symbol R
- Y1: renamed from Y?; value RESONATOR -> 8MHZ_RES
Connections:
- wire segments 121 -> 124
Other:
- moved on the sheet: C5
Changed lines of the file:
@@
 Sheet 1 1
 Title "lipo_arduino_core"
-Date "27 mar 2015"
+Date "27 apr 2015"
 Rev ""
 Comp ""
@@
 L GND #PWR?
 U 1 1 5514EF87
-P 2200 4350
-F 0 "#PWR?" H 2200 4350 30  0001 C CNN
-F 1 "GND" H 2200 4280 30  0001 C CNN
-F 2 "" H 2200 4350 60  0000 C CNN
-F 3 "" H 2200 4350 60  0000 C CNN
-	1    2200 4350
+P 2200 4600
+F 0 "#PWR?" H 2200 4600 30  0001 C CNN
+F 1 "GND" H 2200 4530 30  0001 C CNN
+F 2 "" H 2200 4600 60  0000 C CNN
+F 3 "" H 2200 4600 60  0000 C CNN
+	1    2200 4600
 	1    0    0    -1
 $EndComp
@@
 $EndComp
 $Comp
-L RESONATOR Y?
+L RESONATOR Y1
 U 1 1 5514FCA3
 P 5650 4350
-F 0 "Y?" H 5650 4750 60  0000 C CNN
-F 1 "RESONATOR" H 5650 3950 60  0000 C CNN
+F 0 "Y1" H 5650 4750 60  0000 C CNN
+F 1 "8MHZ_RES" H 5650 3950 60  0000 C CNN
 F 2 "" H 5650 4350 60  0000 C CNN
 F 3 "" H 5650 4350 60  0000 C CNN
@@
 L C C5
 U 1 1 5515CC3D
-P 6100 2700
-F 0 "C5" H 6100 2800 40  0000 L CNN
-F 1 "1uF" H 6106 2615 40  0000 L CNN
-F 2 "~" H 6138 2550 30  0000 C CNN
-F 3 "~" H 6100 2700 60  0000 C CNN
-	1    6100 2700
+P 5500 2600
+F 0 "C5" H 5500 2700 40  0000 L CNN
+F 1 "1uF" H 5506 2515 40  0000 L CNN
+F 2 "~" H 5538 2450 30  0000 C CNN
+F 3 "~" H 5500 2600 60  0000 C CNN
+	1    5500 2600
 	1    0    0    -1
 $EndComp
@@
 	6500 3000 4250 3000
 Wire Wire Line
-	2100 3850 4400 3850
-Wire Wire Line
 	4400 3850 4400 3100
 Wire Wire Line
@@
 	4500 3200 4500 3700
 Wire Wire Line
-	4500 3700 2100 3700
-Wire Wire Line
 	2100 4000 2200 4000
 Wire Wire Line
-	2200 4000 2200 4350
+	2200 4000 2200 4600
 Connection ~ 2200 4150
 Wire Wire Line
@@
 	9200 5600 6400 5600
 Wire Wire Line
-	6150 2300 6500 2300
-Wire Wire Line
-	6150 1250 6150 2500
-Wire Wire Line
 	5700 5000 5700 5500
 Wire Wire Line
@@
 Connection ~ 5000 4350
 Wire Wire Line
-	6500 3300 6100 3300
-Wire Wire Line
-	6100 3300 6100 2900
-Connection ~ 6150 2300
-Connection ~ 6300 2300
-Wire Wire Line
-	6150 2500 6100 2500
-Wire Wire Line
-	6300 2300 6300 2800
-Wire Wire Line
-	6300 2800 6500 2800
-Connection ~ 6300 2700
-Connection ~ 6300 2600
-Connection ~ 6300 2500
-Connection ~ 6300 2400
-Wire Wire Line
-	6500 2400 6300 2400
-Wire Wire Line
-	6300 2500 6500 2500
-Wire Wire Line
-	6500 2600 6300 2600
-Wire Wire Line
-	6300 2700 6500 2700
+	5500 3300 6500 3300
+Wire Wire Line
+	6150 1250 6150 3300
+Wire Wire Line
+	6150 2800 6500 2800
+Connection ~ 6150 2700
+Connection ~ 6150 2600
+Connection ~ 6150 2500
+Connection ~ 6150 2400
+Wire Wire Line
+	6500 2400 6150 2400
+Wire Wire Line
+	6150 2500 6500 2500
+Wire Wire Line
+	6500 2600 6150 2600
+Wire Wire Line
+	6150 2700 6500 2700
 Wire Wire Line
 	5950 3600 5800 3600
@@
 Connection ~ 5200 2250
 Wire Wire Line
-	5500 2100 5500 2250
+	5500 2100 5500 2400
 Wire Wire Line
 	5500 2250 5200 2250
@@
 Wire Wire Line
 	5500 1350 5500 1700
+Connection ~ 2200 4500
+Wire Wire Line
+	800  3550 1000 3550
+Wire Wire Line
+	800  3550 800  4500
+Wire Wire Line
+	800  4500 2200 4500
+Connection ~ 800  3700
+Wire Wire Line
+	1000 3700 800  3700
+$Comp
+L R R4
+U 1 1 553DAAFA
+P 2800 3850
+F 0 "R4" V 2880 3850 40  0000 C CNN
+F 1 "22" V 2807 3851 40  0000 C CNN
+F 2 "~" V 2730 3850 30  0000 C CNN
+F 3 "~" H 2800 3850 30  0000 C CNN
+	1    2800 3850
+	0    1    1    0
+$EndComp
+$Comp
+L R R5
+U 1 1 553DAB15
+P 3300 3700
+F 0 "R5" V 3380 3700 40  0000 C CNN
+F 1 "22" V 3307 3701 40  0000 C CNN
+F 2 "~" V 3230 3700 30  0000 C CNN
+F 3 "~" H 3300 3700 30  0000 C CNN
+	1    3300 3700
+	0    1    1    0
+$EndComp
+Wire Wire Line
+	4400 3850 3050 3850
+Wire Wire Line
+	4500 3700 3550 3700
+Wire Wire Line
+	3050 3700 2100 3700
+Wire Wire Line
+	2550 3850 2100 3850
+Wire Wire Line
+	5500 3300 5500 2800
+Connection ~ 5500 2250
+Connection ~ 6150 3300
+Connection ~ 6150 2800
 $EndSCHEMATC
